File: Front/Front.kicad_sch (KiCad schematic)
At the start: 0 parts

Commit message: a bunch of stuff
Parts:
- added C1, C2, C3, C4, C5, C6, C7: 100nF, Capacitor_THT:C_Disc_D4.7mm_W2.5mm_P5.00mm, symbol Device:C
- added C8: 1µF, Capacitor_THT:CP_Radial_D5.0mm_P2.50mm, symbol Device:C_Polarized
- added D1: A0, LED_THT:LED_D3.0mm, symbol Device:LED_Small
- added D10: A9, LED_THT:LED_D3.0mm, symbol Device:LED_Small
- added D11: A10, LED_THT:LED_D3.0mm, symbol Device:LED_Small
- added D12: A11, LED_THT:LED_D3.0mm, symbol Device:LED_Small
- added D13: A12, LED_THT:LED_D3.0mm, symbol Device:LED_Small
- added D14: A13, LED_THT:LED_D3.0mm, symbol Device:LED_Small
- added D15: A14, LED_THT:LED_D3.0mm, symbol Device:LED_Small
- added D16: A15, LED_THT:LED_D3.0mm, symbol Device:LED_Small
- added D17: D0, LED_THT:LED_D3.0mm_Clear, symbol Device:LED_Small
- added D18: D1, LED_THT:LED_D3.0mm_Clear, symbol Device:LED_Small
- added D19: D2, LED_THT:LED_D3.0mm_Clear, symbol Device:LED_Small
- added D2: A1, LED_THT:LED_D3.0mm, symbol Device:LED_Small
- added D20: D3, LED_THT:LED_D3.0mm_Clear, symbol Device:LED_Small
- added D21: D4, LED_THT:LED_D3.0mm_Clear, symbol Device:LED_Small
- added D22: D5, LED_THT:LED_D3.0mm_Clear, symbol Device:LED_Small
- added D23: D6, LED_THT:LED_D3.0mm_Clear, symbol Device:LED_Small
- added D24: D7, LED_THT:LED_D3.0mm_Clear, symbol Device:LED_Small
- added D25: RAM, LED_THT:LED_D3.0mm, symbol Device:LED_Small
- added D26: ROM, LED_THT:LED_D3.0mm, symbol Device:LED_Small
- added D27: BANK, LED_THT:LED_D3.0mm, symbol Device:LED_Small
- added D28: IO, LED_THT:LED_D3.0mm, symbol Device:LED_Small
- added D29: RESET, LED_THT:LED_D3.0mm, symbol Device:LED_Small
- added D3: A2, LED_THT:LED_D3.0mm, symbol Device:LED_Small
- added D30: NMI, LED_THT:LED_D3.0mm, symbol Device:LED_Small
- added D31: HALT, LED_THT:LED_D3.0mm, symbol Device:LED_Small
- added D32: WRITE, LED_THT:LED_D3.0mm, symbol Device:LED_Small
- added D4: A3, LED_THT:LED_D3.0mm, symbol Device:LED_Small
- added D5: A4, LED_THT:LED_D3.0mm, symbol Device:LED_Small
- added D6: A5, LED_THT:LED_D3.0mm, symbol Device:LED_Small
- added D7: A6, LED_THT:LED_D3.0mm, symbol Device:LED_Small
- added D8: A7, LED_THT:LED_D3.0mm, symbol Device:LED_Small
- added D9: A8, LED_THT:LED_D3.0mm, symbol Device:LED_Small
- added J1: Buss, 0-Footprints:Card, symbol 0-Symbols:Buss
- added J2: Bank, Connector_PinHeader_2.54mm:PinHeader_1x08_P2.54mm_Horizontal, symbol Connector:Conn_01x08_Pin
- added R15: 10K, Resistor_THT:R_Axial_DIN0204_L3.6mm_D1.6mm_P5.08mm_Horizontal, symbol Device:R
- added RN1, RN2, RN3, RN4: 330Ω, Resistor_THT:R_Array_SIP9, symbol Device:R_Network08
- added RN5, RN6: 330Ω, 0-Footprints:Resistor Pack 7, symbol Device:R_Pack07
- added SW1: RESET, Button_Switch_THT:SW_PUSH_6mm, symbol Switch:SW_Push
- added U1, U3: DM9368, Package_DIP:DIP-16_W7.62mm, symbol 0-Symbols:DM9368
- added U10: 74HC14, Package_DIP:DIP-14_W7.62mm, symbol 74xx:74HC14
- added U2: Low Bank, Display_7Segment:HDSP-7401, symbol Display_Character:HDSP-7401
- added U4: High Bank, Display_7Segment:HDSP-7401, symbol Display_Character:HDSP-7401
- added U5, U6, U7: 74LS240, Package_DIP:DIP-20_W7.62mm, symbol 74xx:74LS240
- added U8: 74LS00, Package_DIP:DIP-14_W7.62mm, symbol 74xx:74LS00
- added U9: 74LS245, Package_DIP:DIP-20_W7.62mm, symbol 74xx:74LS245
Connections:
- new net: C8.1, R15.2, SW1.2, U10.1
- new net: D1.1 (K), U5.18 (O0a)
- new net: D1.2 (A), RN1.2 (R1)
- new net: D16.1 (K), U6.3 (O3b)
- new net: D16.2 (A), RN2.9 (R8)
- new net: D17.1 (K), U7.18 (O0a)
- new net: D17.2 (A), RN3.2 (R1)
- new net: RN5.14 (R1.2), U2.10 (A)
- new net: RN5.9 (R6.2), U2.2 (F)
- new net: RN5.8 (R7.2), U2.3 (G)
- new net: RN5.10 (R5.2), U2.4 (E)
- new net: RN5.11 (R4.2), U2.5 (D)
- new net: RN5.12 (R3.2), U2.8 (C)
- new net: RN5.13 (R2.2), U2.9 (B)
- new net: RN5.1 (R1.1), U1.13 (a)
- new net: RN5.2 (R2.1), U1.12 (b)
- new net: RN5.3 (R3.1), U1.11 (c)
- new net: RN5.4 (R4.1), U1.10 (d)
- new net: RN5.5 (R5.1), U1.9 (e)
- new net: RN5.6 (R6.1), U1.15 (f)
- new net: RN5.7 (R7.1), U1.14 (g)
- new net: D21.1 (K), U7.9 (O0b)
- new net: D21.2 (A), RN3.6 (R5)
- new net: D7.1 (K), U5.5 (O2b)
- new net: D7.2 (A), RN1.8 (R7)
- new net: D10.1 (K), U6.16 (O1a)
- new net: D10.2 (A), RN2.3 (R2)
- new net: D9.1 (K), U6.18 (O0a)
- new net: D9.2 (A), RN2.2 (R1)
- new net: U5.1 (OEa), U5.19 (OEb), U6.1 (OEa), U6.19 (OEb), U7.1 (OEa), U7.19 (OEb), U8.3
- new net: D12.1 (K), U6.12 (O3a)
- new net: D11.1 (K), U6.14 (O2a)
- new net: D15.1 (K), U6.5 (O2b)
- new net: D14.1 (K), U6.7 (O1b)
- new net: D13.1 (K), U6.9 (O0b)
- new net: D5.1 (K), U5.9 (O0b)
- new net: D5.2 (A), RN1.6 (R5)
- new net: D22.1 (K), U7.7 (O1b)
- new net: D22.2 (A), RN3.7 (R6)
- new net: D31.1 (K), U9.12 (B6)
- new net: D31.2 (A), RN4.8 (R7)
- new net: D20.1 (K), U7.12 (O3a)
- new net: D20.2 (A), RN3.5 (R4)
- new net: D4.1 (K), U5.12 (O3a)
- new net: D4.2 (A), RN1.5 (R4)
- new net: D28.1 (K), U9.15 (B3)
- new net: D28.2 (A), RN4.5 (R4)
- new net: D19.1 (K), U7.14 (O2a)
- new net: D19.2 (A), RN3.4 (R3)
- new net: D27.1 (K), U9.16 (B2)
- new net: D27.2 (A), RN4.4 (R3)
- new net: D11.2 (A), RN2.4 (R3)
- new net: D12.2 (A), RN2.5 (R4)
- new net: D13.2 (A), RN2.6 (R5)
- new net: D14.2 (A), RN2.7 (R6)
- new net: D15.2 (A), RN2.8 (R7)
- new net: U10.2, U10.3
- new net: D29.1 (K), U9.14 (B4)
- new net: D29.2 (A), RN4.6 (R5)
- new net: D30.1 (K), U9.13 (B5)
- new net: D30.2 (A), RN4.7 (R6)
- new net: D2.1 (K), U5.16 (O1a)
- new net: D2.2 (A), RN1.3 (R2)
- new net: RN6.14 (R1.2), U4.10 (A)
- new net: RN6.9 (R6.2), U4.2 (F)
- new net: RN6.8 (R7.2), U4.3 (G)
- new net: RN6.10 (R5.2), U4.4 (E)
- new net: RN6.11 (R4.2), U4.5 (D)
- new net: RN6.12 (R3.2), U4.8 (C)
- new net: RN6.13 (R2.2), U4.9 (B)
- new net: J2.6 (Pin_6), U3.1 (A1)
- new net: RN6.4 (R4.1), U3.10 (d)
- new net: RN6.3 (R3.1), U3.11 (c)
- new net: RN6.2 (R2.1), U3.12 (b)
- new net: RN6.1 (R1.1), U3.13 (a)
- new net: RN6.7 (R7.1), U3.14 (g)
- new net: RN6.6 (R6.1), U3.15 (f)
- new net: J2.7 (Pin_7), U3.2 (A2)
- new net: J2.8 (Pin_8), U3.6 (A3)
- new net: J2.5 (Pin_5), U3.7 (A0)
- new net: RN6.5 (R5.1), U3.9 (e)
- new net: D24.1 (K), U7.3 (O3b)
- new net: D24.2 (A), RN3.9 (R8)
- new net: D18.1 (K), U7.16 (O1a)
- new net: D18.2 (A), RN3.3 (R2)
- new net: D8.1 (K), U5.3 (O3b)
- new net: D8.2 (A), RN1.9 (R8)
- new net: D3.1 (K), U5.14 (O2a)
- new net: D6.1 (K), U5.7 (O1b)
- new net: D6.2 (A), RN1.7 (R6)
- new net: D26.1 (K), U9.17 (B1)
- new net: D26.2 (A), RN4.3 (R2)
- new net: D23.1 (K), U7.5 (O2b)
- new net: D23.2 (A), RN3.8 (R7)
- new net: D3.2 (A), RN1.4 (R3)
- new net: J2.1 (Pin_1), U1.7 (A0)
- new net: J2.2 (Pin_2), U1.1 (A1)
- new net: J2.3 (Pin_3), U1.2 (A2)
- new net: J2.4 (Pin_4), U1.6 (A3)
- new net: D25.1 (K), U9.18 (B0)
- new net: D25.2 (A), RN4.2 (R1)
- new net: D32.1 (K), U9.11 (B7)
- new net: D32.2 (A), RN4.9 (R8)
- new net +5V: C1.1, C2.1, C3.1, C4.1, C5.1, C6.1, C7.1, J1.P1 (+5V), R15.1, RN1.1 (common), RN2.1 (common), RN3.1 (common), RN4.1 (common), U1.16 (V_{CC}), U1.3 (~{LE}), U10.14 (VCC), U2.1 (CA), U2.6 (CA), U2.7 (DP), U3.16 (V_{CC}), U3.3 (~{LE}), U4.1 (CA), U4.6 (CA), U4.7 (DP), U5.20 (VCC), U6.20 (VCC), U7.20 (VCC), U8.14 (VCC), U9.1 (A->B), U9.20 (VCC)
- new net A0: U5.2 (I0a)
- new net A1: U5.4 (I1a)
- new net A10: U6.6 (I2a)
- new net A11: U6.8 (I3a)
- new net A12: U6.11 (I0b)
- new net A13: U6.13 (I1b)
- new net A14: U6.15 (I2b)
- new net A15: U6.17 (I3b)
- new net A2: U5.6 (I2a)
- new net A3: U5.8 (I3a)
- new net A4: U5.11 (I0b)
- new net A5: U5.13 (I1b)
- new net A6: U5.15 (I2b)
- new net A7: U5.17 (I3b)
- new net A8: U6.2 (I0a)
- new net A9: U6.4 (I1a)
- new net D0: U7.2 (I0a)
- new net D1: U7.4 (I1a)
- new net D2: U7.6 (I2a)
- new net D3: U7.8 (I3a)
- new net D4: U7.11 (I0b)
- new net D5: U7.13 (I1b)
- new net D6: U7.15 (I2b)
- new net D7: U7.17 (I3b)
- new net GND: C1.2, C2.2, C3.2, C4.2, C5.2, C6.2, C7.2, C8.2, J1.P2 (GND), SW1.1, U1.5 (~{RBI}), U1.8 (GND), U10.11, U10.13, U10.5, U10.7 (GND), U10.9, U3.5 (~{RBI}), U3.8 (GND), U5.10 (GND), U6.10 (GND), U7.10 (GND), U8.10, U8.12, U8.13, U8.4, U8.5, U8.7 (GND), U8.9, U9.10 (GND), U9.19 (CE)
- new net R/~{W}: J1.46 (R/~{W}), U9.9 (A7)
- new net VMA: J1.48 (~{IRQ}), J1.B2 (VMA), U8.1
- new net ~{BANK_SEL}: J1.6 (~{BANK_SEL}), U9.4 (A2)
- new net ~{HALT}: J1.B8 (~{HALT}), U9.8 (A6)
- new net ~{IO_SEL}: J1.8 (~{IO_SEL}), U9.5 (A3)
- new net ~{NMI}: J1.B4 (~{NMI}), U9.7 (A5)
- new net ~{RAM_SEL}: J1.2 (~{RAM_SEL}), U9.2 (A0)
- new net ~{RESET}: J1.50 (~{RESET}), U10.4, U9.6 (A4)
- new net ~{ROM_SEL}: J1.4 (~{ROM_SEL}), U9.3 (A1)
- new net Φ2: J1.B3 (Φ2), U8.2
- no-connect marks 0 -> 11
