File: Keyboard/Keyboard.kicad_pcb (KiCad board)
At the start: 2 copper layers, 290.3 x 119.1 mm, 134 parts, among them SW1 Escape, SW10 8/*, SW11 9/(, SW12 0/), SW13 -/_, SW14 =/+, SW15 Delete, SW16 Tab, SW17 Q, SW18 W, SW19 E, SW2 `/~, SW20 R, SW21 T, SW22 Y, SW23 U, SW24 I, SW25 O, SW26 P, SW27 [/{, SW28 ]/}, SW29 \/|, SW3 1/!, SW30 Caps, SW31 A, SW32 S, SW33 D, SW34 F, SW35 G, SW36 H, SW37 J, SW38 K, SW39 L, SW4 2/@, SW40 ;/:, SW41 '/", SW42 Return, SW43 L Shift, SW44 Z, SW45 X, SW46 C, SW47 V, SW48 B, SW49 N, SW5 3/#, SW50 M, SW51 ,/<, SW52 ./>, SW53 //?, SW54 R Shift, SW55 L Control, SW56 L Alt, SW57 L Command, SW58 Space, SW59 R Command, SW6 4/$, SW60 R Alt, SW61 Up, SW62 Left, SW63 Down, SW64 Right, SW65 R Control, SW7 5/%, SW8 6/^, SW9 7/&

Commit message: mostly updating keyboard
Parts:
- added C1: 100nF, 0-Footprints:C_Disc_D5.0mm_W2.5mm_P5.00mm, B.Cu at (150.4, 147.7)
- added C2: 100nF, 0-Footprints:C_Disc_D5.0mm_W2.5mm_P5.00mm, B.Cu at (118.7, 147.7)
- added C3: 100nF, 0-Footprints:C_Disc_D5.0mm_W2.5mm_P5.00mm, B.Cu at (86.9, 147.7)
- added G1: Logo, 0-Footprints:Crank, F.Cu at (187.3, 149.7)
- added G2: Logo, Symbol:OSHW-Logo2_7.3x6mm_SilkScreen, F.Cu at (251.2, 149.7)
- added G3: Logo, 0-Footprints:crankery_small, F.Cu at (234.5, 149.8)
- added H10: MountingHole, 0-Footprints:MountingHole_2.1mm, F.Cu at (203.7, 159.2)
- added H11: MountingHole, 0-Footprints:MountingHole_2.1mm, F.Cu at (260.8, 44.8)
- added H12: MountingHole, 0-Footprints:MountingHole_2.1mm, F.Cu at (260.8, 159.2)
- added H13: MountingHole, 0-Footprints:MountingHole_2.1mm, F.Cu at (32.2, 102.0)
- added H14: MountingHole, 0-Footprints:MountingHole_2.1mm, F.Cu at (94.1, 102.0)
- added H15: MountingHole, 0-Footprints:MountingHole_2.1mm, F.Cu at (151.2, 102.0)
- added H16: MountingHole, 0-Footprints:MountingHole_2.1mm, F.Cu at (208.4, 102.0)
- added H17: MountingHole, 0-Footprints:MountingHole_2.1mm, F.Cu at (265.5, 102.0)
- added H18: MountingHole, 0-Footprints:MountingHole_2.1mm, F.Cu at (317.9, 102.0)
- added H5: MountingHole, 0-Footprints:MountingHole_2.1mm, F.Cu at (89.4, 44.8)
- added H6: MountingHole, 0-Footprints:MountingHole_2.1mm, F.Cu at (75.9, 159.2)
- added H7: MountingHole, 0-Footprints:MountingHole_2.1mm, F.Cu at (146.6, 44.8)
- added H8: MountingHole, 0-Footprints:MountingHole_2.1mm, F.Cu at (146.6, 159.2)
- added H9: MountingHole, 0-Footprints:MountingHole_2.1mm, F.Cu at (203.7, 44.8)
- added J1: Keyboard, 0-Footprints:PinHeader_1x09_P2.54mm_Horizontal, B.Cu at (50.7, 144.5)
- added R12: 220Ω, Resistor_THT:R_Axial_DIN0204_L3.6mm_D1.6mm_P7.62mm_Horizontal, B.Cu at (36.8, 88.6)
- added RN1: 4.7K, Resistor_THT:R_Array_SIP5, B.Cu at (137.7, 157.8)
- added RN2: 4.7K, Resistor_THT:R_Array_SIP5, B.Cu at (125.0, 142.5)
- added RN3: 4.7K, Resistor_THT:R_Array_SIP5, B.Cu at (169.5, 157.8)
- added U1: 74LS138, 0-Footprints:DIP-16_W7.62mm, B.Cu at (90.7, 146.3)
- added U2: 74LS165, 0-Footprints:DIP-16_W7.62mm, B.Cu at (122.5, 146.3)
- added U3: 74LS165, 0-Footprints:DIP-16_W7.62mm, B.Cu at (154.3, 146.3)
- D10, D11, D12, D13, D14, D16, D17, D18, D19, D2, D20, D21, D22, D23, D24, D25, D26, D27, D28, D3, D30, D31, D32, D33, D34, D35, D36, D37, D38, D39, D4, D40, D41, D42, D44, D45, D46, D47, D48, D49, D5, D50, D51, D52, D53, D54, D55, D56, D58, D59, D6, D60, D61, D62, D63, D64, D65, D66, D67, D68, D69, D7, D70, D8, D9: footprint Diode_THT:D_DO-35_SOD27_P7.62mm_Horizontal -> 0-Footprints:D_DO-35_SOD27_P7.62mm_Horizontal; moved to B.Cu
- SW30: footprint 0-Footprints:SW_Cherry_MX_1.75u_PCB -> 0-Footprints:SW_Cherry_MX_1.75u_PCB_LED
- moved D69 7.81 mm to (282.2, 107.7), turned to -90 degrees
- moved D2 7.73 mm to (32.2, 50.5), turned to -90 degrees
- moved D42 7.73 mm to (289.3, 50.5), turned to -90 degrees
- moved D44 7.73 mm to (44.1, 107.7), turned to -90 degrees
- moved D54 7.73 mm to (246.5, 107.7), turned to -90 degrees
- moved D55 7.73 mm to (294.1, 69.6), turned to -90 degrees
- moved D56 7.73 mm to (287.0, 88.6), turned to -90 degrees
- moved D58 7.73 mm to (34.6, 126.8), turned to -90 degrees
- moved D59 7.73 mm to (58.4, 126.8), turned to -90 degrees
- moved D60 7.73 mm to (82.2, 126.8), turned to -90 degrees
- moved D61 7.73 mm to (153.6, 126.8), turned to -90 degrees
- moved D62 7.73 mm to (222.7, 126.8), turned to -90 degrees
- moved D63 7.73 mm to (241.7, 126.8), turned to -90 degrees
- moved D66 7.73 mm to (260.8, 145.9), turned to -90 degrees
- moved D67 7.73 mm to (279.8, 145.9), turned to -90 degrees
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Connections:
- D10 pad 1: unconnected-(D10-K-Pad1) -> Net-(D10-K)
- D10 pad 2: Net-(D10-A) -> /R0
- D11 pad 1: unconnected-(D11-K-Pad1) -> Net-(D11-K)
- D11 pad 2: Net-(D11-A) -> /R0
- D12 pad 1: unconnected-(D12-K-Pad1) -> Net-(D12-K)
- D12 pad 2: Net-(D12-A) -> /R0
- D13 pad 1: unconnected-(D13-K-Pad1) -> Net-(D13-K)
- D13 pad 2: Net-(D13-A) -> /R5
- D14 pad 1: unconnected-(D14-K-Pad1) -> Net-(D14-K)
- D14 pad 2: Net-(D14-A) -> /R5
- D16 pad 2: Net-(D16-A) -> /R1
- D17 pad 2: Net-(D17-A) -> /R1
- D18 pad 2: Net-(D18-A) -> /R1
- D19 pad 2: Net-(D19-A) -> /R1
- D2 pad 1: unconnected-(D2-K-Pad1) -> Net-(D2-K)
- D2 pad 2: Net-(D16-K) -> /R0
- D20 pad 2: Net-(D20-A) -> /R1
- D21 pad 2: Net-(D21-A) -> /R1
- D22 pad 2: Net-(D22-A) -> /R1
- D23 pad 2: Net-(D23-A) -> /R1
- D24 pad 1: Net-(D10-A) -> Net-(D24-K)
- D24 pad 2: Net-(D24-A) -> /R1
- D25 pad 1: Net-(D11-A) -> Net-(D25-K)
- D25 pad 2: Net-(D25-A) -> /R1
- D26 pad 1: Net-(D12-A) -> Net-(D26-K)
- D26 pad 2: Net-(D26-A) -> /R1
- D27 pad 1: Net-(D13-A) -> Net-(D27-K)
- D27 pad 2: Net-(D27-A) -> /R5
- D28 pad 1: Net-(D14-A) -> Net-(D28-K)
- D28 pad 2: Net-(D28-A) -> /R5
- D3 pad 1: unconnected-(D3-K-Pad1) -> Net-(D3-K)
- D3 pad 2: Net-(D17-K) -> /R0
- D30 pad 1: Net-(D16-A) -> Net-(D30-K)
- D30 pad 2: Net-(D30-A) -> /R2
- D31 pad 1: Net-(D17-A) -> Net-(D31-K)
- D31 pad 2: Net-(D31-A) -> /R2
- D32 pad 1: Net-(D18-A) -> Net-(D32-K)
- D32 pad 2: Net-(D32-A) -> /R2
- D33 pad 1: Net-(D19-A) -> Net-(D33-K)
- D33 pad 2: Net-(D33-A) -> /R2
- D34 pad 1: Net-(D20-A) -> Net-(D34-K)
- D34 pad 2: Net-(D34-A) -> /R2
- D35 pad 1: Net-(D21-A) -> Net-(D35-K)
- D35 pad 2: Net-(D35-A) -> /R2
- D36 pad 1: Net-(D22-A) -> Net-(D36-K)
- D36 pad 2: Net-(D36-A) -> /R2
- D37 pad 1: Net-(D23-A) -> Net-(D37-K)
- D37 pad 2: Net-(D37-A) -> /R2
- D38 pad 1: Net-(D24-A) -> Net-(D38-K)
- D38 pad 2: Net-(D38-A) -> /R2
- D39 pad 1: Net-(D25-A) -> Net-(D39-K)
- D39 pad 2: Net-(D39-A) -> /R2
- D4 pad 1: unconnected-(D4-K-Pad1) -> Net-(D4-K)
- D4 pad 2: Net-(D18-K) -> /R0
- D40 pad 1: Net-(D26-A) -> Net-(D40-K)
- D40 pad 2: Net-(D40-A) -> /R2
- D41 pad 1: Net-(D27-A) -> Net-(D41-K)
- D41 pad 2: Net-(D41-A) -> /R5
- D42 pad 1: Net-(D28-A) -> Net-(D42-K)
- D42 pad 2: Net-(D42-A) -> /R5
- D44 pad 1: Net-(D30-A) -> Net-(D44-K)
- D44 pad 2: Net-(D44-A) -> /R3
- D45 pad 1: Net-(D31-A) -> Net-(D45-K)
- D45 pad 2: Net-(D45-A) -> /R3
- D46 pad 1: Net-(D32-A) -> Net-(D46-K)
- D46 pad 2: Net-(D46-A) -> /R3
- D47 pad 1: Net-(D33-A) -> Net-(D47-K)
- D47 pad 2: Net-(D47-A) -> /R3
- D48 pad 1: Net-(D34-A) -> Net-(D48-K)
- D48 pad 2: Net-(D48-A) -> /R3
- D49 pad 1: Net-(D35-A) -> Net-(D49-K)
- D49 pad 2: Net-(D49-A) -> /R3
- D5 pad 1: unconnected-(D5-K-Pad1) -> Net-(D5-K)
- D5 pad 2: Net-(D19-K) -> /R0
- D50 pad 1: Net-(D36-A) -> Net-(D50-K)
- D50 pad 2: Net-(D50-A) -> /R3
- D51 pad 1: Net-(D37-A) -> Net-(D51-K)
- D51 pad 2: Net-(D51-A) -> /R3
- D52 pad 1: Net-(D38-A) -> Net-(D52-K)
- D52 pad 2: Net-(D52-A) -> /R3
- D53 pad 1: Net-(D39-A) -> Net-(D53-K)
- D53 pad 2: Net-(D53-A) -> /R3
- D54 pad 1: Net-(D40-A) -> Net-(D54-K)
- D54 pad 2: Net-(D54-A) -> /R3
- D55 pad 1: Net-(D41-A) -> Net-(D55-K)
- D55 pad 2: Net-(D55-A) -> /R5
- D56 pad 1: unconnected-(D56-K-Pad1) -> Net-(D56-K)
- D56 pad 2: Net-(D56-A) -> /R5
- D58 pad 1: Net-(D44-A) -> Net-(D58-K)
- D58 pad 2: Net-(D58-A) -> /R4
- D59 pad 1: Net-(D45-A) -> Net-(D59-K)
- D59 pad 2: Net-(D59-A) -> /R4
- D6 pad 1: unconnected-(D6-K-Pad1) -> Net-(D6-K)
- D6 pad 2: Net-(D20-K) -> /R0
- D60 pad 1: Net-(D46-A) -> Net-(D60-K)
- D60 pad 2: Net-(D60-A) -> /R4
- D61 pad 1: Net-(D47-A) -> Net-(D61-K)
- D61 pad 2: Net-(D61-A) -> /R4
- D62 pad 1: Net-(D48-A) -> Net-(D62-K)
- D62 pad 2: Net-(D62-A) -> /R4
- D63 pad 1: Net-(D49-A) -> Net-(D63-K)
- D63 pad 2: Net-(D63-A) -> /R4
- D64 pad 1: Net-(D50-A) -> Net-(D64-K)
- D64 pad 2: Net-(D64-A) -> /R4
- D65 pad 1: Net-(D51-A) -> Net-(D65-K)
- D65 pad 2: Net-(D65-A) -> /R4
- D66 pad 1: Net-(D52-A) -> Net-(D66-K)
- D66 pad 2: Net-(D66-A) -> /R4
- D67 pad 1: Net-(D53-A) -> Net-(D67-K)
- D67 pad 2: Net-(D67-A) -> /R4
- D68 pad 1: Net-(D54-A) -> Net-(D68-K)
- D68 pad 2: Net-(D68-A) -> /R4
- D69 pad 1: Net-(D55-A) -> Net-(D69-K)
- D69 pad 2: Net-(D69-A) -> /R5
- D7 pad 1: unconnected-(D7-K-Pad1) -> Net-(D7-K)
- D7 pad 2: Net-(D21-K) -> /R0
- D70 pad 1: Net-(D56-A) -> Net-(D70-K)
- D70 pad 2: Net-(D70-A) -> /R5
- D8 pad 1: unconnected-(D8-K-Pad1) -> Net-(D8-K)
- D8 pad 2: Net-(D22-K) -> /R0
- D9 pad 1: unconnected-(D9-K-Pad1) -> Net-(D9-K)
- D9 pad 2: Net-(D23-K) -> /R0
- SW1 pad 1: Net-(SW1-Pad1) -> Net-(D2-K)
- SW1 pad 2: Net-(D16-K) -> /C0
- SW10 pad 1: Net-(SW1-Pad1) -> Net-(D10-K)
- SW10 pad 2: Net-(D10-A) -> /C8
- SW11 pad 1: Net-(SW1-Pad1) -> Net-(D11-K)
- SW11 pad 2: Net-(D11-A) -> /C9
- SW12 pad 1: Net-(SW1-Pad1) -> Net-(D12-K)
- SW12 pad 2: Net-(D12-A) -> /C10
- SW13 pad 1: Net-(SW1-Pad1) -> Net-(D13-K)
- SW13 pad 2: Net-(D13-A) -> /C5
- SW14 pad 1: Net-(SW1-Pad1) -> Net-(D14-K)
- SW14 pad 2: Net-(D14-A) -> /C0
- SW15 pad 1: Net-(SW15-Pad1) -> Net-(D42-K)
- SW15 pad 2: Net-(D42-A) -> /C2
- SW16 pad 1: Net-(SW16-Pad1) -> Net-(D16-K)
- SW16 pad 2: Net-(D16-A) -> /C0
- SW17 pad 1: Net-(SW16-Pad1) -> Net-(D17-K)
- SW17 pad 2: Net-(D17-A) -> /C1
- SW18 pad 1: Net-(SW16-Pad1) -> Net-(D18-K)
- SW18 pad 2: Net-(D18-A) -> /C2
- SW19 pad 1: Net-(SW16-Pad1) -> Net-(D19-K)
- SW19 pad 2: Net-(D19-A) -> /C3
- SW2 pad 1: Net-(SW2-Pad1) -> Net-(D70-K)
- SW2 pad 2: Net-(D70-A) -> /C4
- SW20 pad 1: Net-(SW16-Pad1) -> Net-(D20-K)
- SW20 pad 2: Net-(D20-A) -> /C4
- SW21 pad 1: Net-(SW16-Pad1) -> Net-(D21-K)
- SW21 pad 2: Net-(D21-A) -> /C5
- SW22 pad 1: Net-(SW16-Pad1) -> Net-(D22-K)
- SW22 pad 2: Net-(D22-A) -> /C6
- SW23 pad 1: Net-(SW16-Pad1) -> Net-(D23-K)
- SW23 pad 2: Net-(D23-A) -> /C7
- SW24 pad 1: Net-(SW16-Pad1) -> Net-(D24-K)
- SW24 pad 2: Net-(D24-A) -> /C8
- SW25 pad 1: Net-(SW16-Pad1) -> Net-(D25-K)
- SW25 pad 2: Net-(D25-A) -> /C9
- SW26 pad 1: unconnected-(SW26-Pad1) -> Net-(D26-K)
- SW26 pad 2: Net-(D26-A) -> /C10
- SW27 pad 1: Net-(SW16-Pad1) -> Net-(D27-K)
- SW27 pad 2: Net-(D27-A) -> /C6
- SW28 pad 1: Net-(SW16-Pad1) -> Net-(D28-K)
- SW28 pad 2: Net-(D28-A) -> /C1
- SW29 pad 1: unconnected-(SW29-Pad1) -> Net-(D55-K)
- SW29 pad 2: Net-(D55-A) -> /C8
- SW3 pad 1: Net-(SW1-Pad1) -> Net-(D3-K)
- SW3 pad 2: Net-(D17-K) -> /C1
- SW30 pad 1: Net-(SW15-Pad1) -> Net-(D30-K)
- SW30 pad 2: Net-(D30-A) -> /C0
- SW31 pad 1: Net-(SW15-Pad1) -> Net-(D31-K)
- SW31 pad 2: Net-(D31-A) -> /C1
- SW32 pad 1: Net-(SW15-Pad1) -> Net-(D32-K)
- SW32 pad 2: Net-(D32-A) -> /C2
- SW33 pad 1: Net-(SW15-Pad1) -> Net-(D33-K)
- SW33 pad 2: Net-(D33-A) -> /C3
- SW34 pad 1: Net-(SW15-Pad1) -> Net-(D34-K)
- SW34 pad 2: Net-(D34-A) -> /C4
- SW35 pad 1: Net-(SW15-Pad1) -> Net-(D35-K)
- SW35 pad 2: Net-(D35-A) -> /C5
- SW36 pad 1: Net-(SW15-Pad1) -> Net-(D36-K)
- SW36 pad 2: Net-(D36-A) -> /C6
- SW37 pad 1: Net-(SW15-Pad1) -> Net-(D37-K)
- SW37 pad 2: Net-(D37-A) -> /C7
- SW38 pad 1: Net-(SW15-Pad1) -> Net-(D38-K)
- SW38 pad 2: Net-(D38-A) -> /C8
- SW39 pad 1: Net-(SW15-Pad1) -> Net-(D39-K)
- SW39 pad 2: Net-(D39-A) -> /C9
- SW4 pad 1: Net-(SW1-Pad1) -> Net-(D4-K)
- SW4 pad 2: Net-(D18-K) -> /C2
- SW40 pad 1: Net-(SW15-Pad1) -> Net-(D40-K)
- SW40 pad 2: Net-(D40-A) -> /C10
- SW41 pad 1: Net-(SW15-Pad1) -> Net-(D41-K)
- SW41 pad 2: Net-(D41-A) -> /C7
- SW42 pad 1: Net-(SW42-Pad1) -> Net-(D56-K)
- SW42 pad 2: Net-(D56-A) -> /C3
- SW43 pad 1: Net-(SW42-Pad1) -> Net-(D44-K)
- SW43 pad 2: Net-(D44-A) -> /C0
- SW44 pad 1: Net-(SW42-Pad1) -> Net-(D45-K)
- SW44 pad 2: Net-(D45-A) -> /C1
- SW45 pad 1: Net-(SW42-Pad1) -> Net-(D46-K)
- SW45 pad 2: Net-(D46-A) -> /C2
- SW46 pad 1: Net-(SW42-Pad1) -> Net-(D47-K)
- SW46 pad 2: Net-(D47-A) -> /C3
- SW47 pad 1: Net-(SW42-Pad1) -> Net-(D48-K)
- SW47 pad 2: Net-(D48-A) -> /C4
- SW48 pad 1: Net-(SW42-Pad1) -> Net-(D49-K)
- SW48 pad 2: Net-(D49-A) -> /C5
- SW49 pad 1: Net-(SW42-Pad1) -> Net-(D50-K)
- SW49 pad 2: Net-(D50-A) -> /C6
- SW5 pad 1: Net-(SW1-Pad1) -> Net-(D5-K)
- SW5 pad 2: Net-(D19-K) -> /C3
- SW50 pad 1: Net-(SW42-Pad1) -> Net-(D51-K)
- SW50 pad 2: Net-(D51-A) -> /C7
- SW51 pad 1: Net-(SW42-Pad1) -> Net-(D52-K)
- SW51 pad 2: Net-(D52-A) -> /C8
- SW52 pad 1: Net-(SW42-Pad1) -> Net-(D53-K)
- SW52 pad 2: Net-(D53-A) -> /C9
- SW53 pad 1: Net-(SW42-Pad1) -> Net-(D54-K)
- SW53 pad 2: Net-(D54-A) -> /C10
- SW54 pad 1: Net-(SW2-Pad1) -> Net-(D69-K)
- SW54 pad 2: Net-(D69-A) -> /C9
- SW55 pad 1: Net-(SW2-Pad1) -> Net-(D58-K)
- SW55 pad 2: Net-(D58-A) -> /C0
- SW56 pad 1: Net-(SW2-Pad1) -> Net-(D59-K)
- SW56 pad 2: Net-(D59-A) -> /C1
- SW57 pad 1: Net-(SW2-Pad1) -> Net-(D60-K)
- SW57 pad 2: Net-(D60-A) -> /C2
- SW58 pad 1: Net-(SW2-Pad1) -> Net-(D61-K)
- SW58 pad 2: Net-(D61-A) -> /C3
- SW59 pad 1: Net-(SW2-Pad1) -> Net-(D62-K)
- SW59 pad 2: Net-(D62-A) -> /C4
- SW6 pad 1: Net-(SW1-Pad1) -> Net-(D6-K)
- SW6 pad 2: Net-(D20-K) -> /C4
- SW60 pad 1: Net-(SW2-Pad1) -> Net-(D63-K)
- SW60 pad 2: Net-(D63-A) -> /C5
- SW61 pad 1: Net-(SW2-Pad1) -> Net-(D65-K)
- SW61 pad 2: Net-(D65-A) -> /C7
- SW62 pad 1: Net-(SW2-Pad1) -> Net-(D66-K)
- SW62 pad 2: Net-(D66-A) -> /C8
- SW63 pad 1: Net-(SW2-Pad1) -> Net-(D67-K)
- SW63 pad 2: Net-(D67-A) -> /C9
- SW64 pad 1: Net-(SW2-Pad1) -> Net-(D68-K)
- SW64 pad 2: Net-(D68-A) -> /C10
- SW65 pad 1: Net-(SW2-Pad1) -> Net-(D64-K)
- SW65 pad 2: Net-(D64-A) -> /C6
- SW7 pad 1: Net-(SW1-Pad1) -> Net-(D7-K)
- SW7 pad 2: Net-(D21-K) -> /C5
- SW8 pad 1: Net-(SW1-Pad1) -> Net-(D8-K)
- SW8 pad 2: Net-(D22-K) -> /C6
- SW9 pad 1: Net-(SW1-Pad1) -> Net-(D9-K)
- SW9 pad 2: Net-(D23-K) -> /C7
Routing:
- net /C0: track 0.00 -> 438.2 mm, vias 0 -> 2
- net /R5: track 0.00 -> 424.6 mm, vias 0 -> 4
- net /C1: track 0.00 -> 405.1 mm, vias 0 -> 2
- net /C2: track 0.00 -> 386.8 mm, vias 0 -> 2
- net /C3: track 0.00 -> 361.0 mm, vias 0 -> 3
- net /C5: track 0.00 -> 344.5 mm, vias 0 -> 3
- net /R4: track 0.00 -> 323.4 mm, vias 0 -> 1
- net /C8: track 0.00 -> 319.5 mm, vias 0 -> 1
- net /C6: track 0.00 -> 303.4 mm, vias 0 -> 2
- net /C7: track 0.00 -> 299.1 mm, vias 0 -> 4
- net /R0: track 0.00 -> 296.3 mm
- net /C4: track 0.00 -> 280.6 mm, vias 0 -> 1
- net /R1: track 0.00 -> 279.0 mm, vias 0 -> 1
- net /C9: track 0.00 -> 275.5 mm, vias 0 -> 1
- net /R2: track 0.00 -> 257.5 mm
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- added copper zone on B.Cu, net GND
- added copper zone on F.Cu, net GND
Other:
- outline, holes or cut-outs redrawn
- board text added: "C68KB.01"
- board text added: "JLCJLCJLCJLC"
