File: Math/Math.kicad_sch (KiCad schematic)
At the start: 7 parts, among them J1 Buss, SW1 Slot, U1 AM9511A, U2 74LS85, U3 74LS04, U4 74LS30

Commit message: mainly actually saving out vs.code along with sorting out the math card
Parts:
- removed U3: 74LS04, Package_DIP:DIP-14_W7.62mm, symbol 74xx:74LS04
- removed U4: 74LS30, Package_DIP:DIP-14_W7.62mm, symbol 74xx:74LS30
- added C1, C2, C3, C4, C5: 100nF, 0-Footprints:C_Disc_D5.0mm_W2.5mm_P5.00mm, symbol Device:C
- added G1: Logo, 0-Footprints:Crank, symbol 0-Symbols:Logo
- added G2: Logo, 0-Footprints:crankery_small, symbol 0-Symbols:Logo
- added JP1: ~{EACK}, 0-Footprints:SolderJumper-2_P1.3mm_Bridged_RoundedPad1.0x1.5mm, symbol Jumper:SolderJumper_2_Bridged
- added JP2: ~{SVACK}, 0-Footprints:SolderJumper-2_P1.3mm_Bridged_RoundedPad1.0x1.5mm, symbol Jumper:SolderJumper_2_Bridged
- added QC1, QC2, QC3: Grid, 0-Footprints:Grid, symbol 0-Symbols:Grid
- added TP1: ~{EACK}, 0-Footprints:TestPoint_THTPad_D1.5mm_Drill0.7mm, symbol Connector:TestPoint
- added TP2: ~{SVACK}, 0-Footprints:TestPoint_THTPad_D1.5mm_Drill0.7mm, symbol Connector:TestPoint
- added TP3: ~{END}, 0-Footprints:TestPoint_THTPad_D1.5mm_Drill0.7mm, symbol Connector:TestPoint
- added TP4: ~{PAUSE}, 0-Footprints:TestPoint_THTPad_D1.5mm_Drill0.7mm, symbol Connector:TestPoint
- added TP5: ~{SVREQ}, 0-Footprints:TestPoint_THTPad_D1.5mm_Drill0.7mm, symbol Connector:TestPoint
- added TP6: ~{CS} AM9511, 0-Footprints:TestPoint_THTPad_D1.5mm_Drill0.7mm, symbol Connector:TestPoint
- added U3: 74LS00, 0-Footprints:DIP-14_W7.62mm, symbol 74xx:74LS00
- added U4: 74LS139, 0-Footprints:DIP-16_W7.62mm, symbol 74xx:74LS139
- added Y1: 2.000MHz, 0-Footprints:Oscillator_DIP-14, symbol Oscillator:ACO-xxxMHz
- RN1: footprint Resistor_THT:R_Array_SIP5 -> 0-Footprints:R_Array_SIP5
- SW1: footprint (none) -> 0-Footprints:SW_DIP_SPSTx04_Slide_9.78x12.34mm_W7.62mm_P2.54mm
- U1: footprint Package_DIP:DIP-24_18.0mmx34.29mm_W15.24mm -> 0-Footprints:DIP-24_W15.24mm
- U2: footprint Package_DIP:DIP-16_W7.62mm -> 0-Footprints:DIP-16_W7.62mm
Connections:
- net +12V: now also J1.P3 (+12V), C1.1; no longer J1.VCC (-12V)
- net +5V: now also J1.P1 (+5V), C2.1, C3.1, C4.1, C5.2, JP1.2 (B), JP2.2 (B), QC1.1 (VCC), QC2.1 (VCC), QC3.1 (VCC), U3.14 (VCC), U4.16 (VCC), Y1.14 (Vcc); no longer J1.VCC (-12V), U1.3 (~{EACK}), U1.4 (~{SVACK})
- net A1: now also U4.14 (A0)
- net A2: now also U4.13 (A1)
- net A3: now also U4.2 (A0)
- net BUS_OK: now also U3.9
- net GND: now also J1.P2 (GND), C1.2, C2.2, C3.2, C4.2, C5.1, QC1.2 (GND), QC2.2 (GND), QC3.2 (GND), U3.12, U3.13, U3.7 (GND), U4.8 (GND), Y1.7 (GND); no longer J1.GND
- net R/~{W}: now also U3.4, U3.5
- net SLOT_SEL: now also U3.10
- net ~{IO_SEL}: now also U4.1 (E)
- net ~{RESET}: now also U3.1, U3.2
- net ~{PAUSE}: now reaches U1.17 (~{PAUSE})
- net ~{PAUSE}: now also TP4.1
- net at U1.22 (RESET): now also U3.3
- net ~{END}: now reaches U1.24 (~{END})
- net ~{END}: now also TP3.1
- net SVREQ: now reaches U1.5 (SVREQ)
- net SVREQ: now also TP5.1
- net W/~{R}: no longer names the net of U1.20 (~{RD})
- net W/~{R}: now also U3.6
- net ~{CS_AM9511} renamed ~{CS_9511}
- net ~{CS_9511}: now also TP6.1, U4.12 (O0)
- net Φ2: no longer names the net of U1.23 (CLK)
- net Φ2: now also Y1.8 (OUT); no longer J1.B3 (Φ2)
- new net: U3.8, U4.3 (A1)
- new net: U4.15 (E), U4.4 (O0)
- new net ~{EACK}: JP1.1 (A), TP1.1, U1.3 (~{EACK})
- new net ~{SVACK}: JP2.1 (A), TP2.1, U1.4 (~{SVACK})
- no-connect marks 20 -> 24
