File: BankedMemory/BankedMemory.kicad_sch (KiCad schematic)
At the start: 24 parts, among them J1 Buss, U1 AS6C4008_{0}, U2 AS6C4008_{1}, U3 74LS00, U4 GAL22V10, U5 74LS573, U6 DS1210, U7 DS1210

Commit message: finish routing the coms board. add some step models to look at this thing in freecad
Parts:
- removed U3: 74LS00, Package_DIP:DIP-14_W7.62mm, symbol 74xx:74LS00
- added G1: Logo, 0-Footprints:Crank, symbol 0-Symbols:Logo
- added G2: Logo, 0-Footprints:crankery_small, symbol 0-Symbols:Logo
- added U3: 74LS573, 0-Footprints:DIP-20_W7.62mm, symbol 74xx:74LS573
- BT1: footprint Battery:BatteryHolder_Keystone_1060_1x2032 -> 0-Footprints:BatteryHolder_Keystone_1060_1x2032
- C1, C11, C2, C3, C4, C5, C6, C8, C9: value 100n -> 100nF; footprint Capacitor_THT:C_Disc_D3.0mm_W1.6mm_P2.50mm -> 0-Footprints:C_Disc_D5.0mm_W2.5mm_P5.00mm
- C10, C7: footprint Capacitor_THT:CP_Radial_D5.0mm_P2.50mm -> 0-Footprints:CP_Radial_D5.0mm_P2.50mm
- J1: value Buss -> Card
- JP1, JP3: value BE -> Low
- JP2, JP4: value BE -> High
- U1, U2: footprint Package_DIP:DIP-32_W15.24mm -> 0-Footprints:DIP-32_W15.24mm
- U4: footprint Package_DIP:DIP-24_W7.62mm -> 0-Footprints:DIP-24_W7.62mm
- U5: footprint Package_DIP:DIP-20_W7.62mm -> 0-Footprints:DIP-20_W7.62mm
- U6, U7: footprint Package_DIP:DIP-8_W7.62mm -> 0-Footprints:DIP-8_W7.62mm
Connections:
- net +5V_{B} is gone; now on net GND: C5.2
- net ~{BANK_SEL_{0}_B} is gone; now on net ~{BANK_{LB}}: JP3.1 (A)
- net ~{BANK_SEL_{0}} is gone; now on net ~{BANK_{L}}: JP3.3 (B)
- net ~{BANK_SEL_{1}_B} is gone; now on net ~{BANK_{HB}}: JP4.1 (A)
- net ~{BANK_SEL_{1}} is gone; now on net ~{BANK_{H}}: JP4.3 (B)
- net +5V: now also C5.1, J1.P1 (+5V), U3.20 (VCC); no longer J1.VCC (-12V)
- net A12: now also U4.23 (I/0); no longer U1.4 (A12), U2.4 (A12)
- net BANK_0: now also U1.4 (A12), U2.4 (A12), U3.12 (Q7); no longer U1.28 (A13), U2.28 (A13)
- net BANK_1: now also U1.28 (A13), U2.28 (A13), U3.13 (Q6); no longer U1.3 (A14), U2.3 (A14)
- net BANK_2: now also U1.3 (A14), U2.3 (A14), U3.14 (Q5); no longer U1.31 (A15), U2.31 (A15)
- net BANK_3: now also U1.31 (A15), U2.31 (A15), U3.15 (Q4); no longer U1.2 (A16), U2.2 (A16)
- net BANK_4: now also U1.2 (A16), U2.2 (A16), U3.16 (Q3); no longer U1.30 (A17), U2.30 (A17)
- net BANK_5: now also U1.30 (A17), U2.30 (A17), U3.17 (Q2); no longer U1.1 (A18), U2.1 (A18)
- net BANK_6: now also U1.1 (A18), U2.1 (A18), U3.18 (Q1)
- net BANK_7: now also U3.19 (Q0)
- net D0: now also U3.9 (D7)
- net D1: now also U3.8 (D6)
- net D2: now also U3.7 (D5)
- net D3: now also U3.6 (D4)
- net D4: now also U3.5 (D3)
- net D5: now also U3.4 (D2)
- net D6: now also U3.3 (D1)
- net D7: now also U3.2 (D0)
- net GND: now also J1.P2 (GND), U3.10 (GND); no longer C5.1, J1.GND, U4.17 (I/O), U4.18 (I/O), U4.19 (I/O), U4.20 (I/O), U5.1 (OE)
- net ~{OE}: now also U4.22 (I/O); no longer U4.23 (I/0)
- net ~{WE}: now also U4.21 (I/O); no longer U4.22 (I/O)
- net +5V_{B1} renamed +5V_{LB}
- net +5V_{B2} renamed +5V_{HB}
- net A13: no longer names the net of J1.27 (A_{13})
- net A14: no longer names the net of J1.29 (A_{14})
- net A15: no longer names the net of J1.31 (A_{15})
- net LOAD_LATCH renamed LOAD_{L}
- net LOAD_{L}: now also U4.20 (I/O); no longer U4.21 (I/O)
- net ~{BANK_CS_{0}_B} renamed ~{BANK_{LB}}
- net ~{BANK_CS_{0}} renamed ~{BANK_{L}}
- net ~{BANK_{L}}: now also U4.18 (I/O), U5.1 (OE)
- net ~{BANK_CS_{1}_B} renamed ~{BANK_{HB}}
- net ~{BANK_CS_{1}} renamed ~{BANK_{H}}
- net ~{BANK_{H}}: now also U4.17 (I/O), U3.1 (OE)
- new net LOAD_{H}: U3.11 (Load), U4.19 (I/O)
- no-connect marks 3 -> 33
Other:
- note added: "~{OE}: BUS_OK && !~{BANK_SEL} && R/~{W} ~{WE}: BUS_OK && !~{BANK_SEL} && !R/~{W} LOAD_{L}: BUS_OK && !~{IO_SEL} && !A0 && ![A1..A7] && !R/~{W} LOAD_{H}: BUS_OK && !~{IO_SEL} && A0 && ![A1..A7] && !R/~{W} ~{BANK_{L}}: BUS_OK && !~{IO_SEL} & !A12 ~{BANK_{H}}: BUS_OK && !~{IO_SEL} & A12"
- moved on the sheet: BT1, C10, C11, C3, C4, C6, C7, C8, C9, U4, U5, U6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

Commit message: lots of fixes to stack handling on emu, fix the latches on the banked memory board, tons of little bug fixes
Parts:
- removed JP1, JP3: Low, Jumper:SolderJumper-3_P1.3mm_Bridged12_RoundedPad1.0x1.5mm, symbol Jumper:Jumper_3_Bridged12
- removed JP2, JP4: High, Jumper:SolderJumper-3_P1.3mm_Bridged12_RoundedPad1.0x1.5mm, symbol Jumper:Jumper_3_Bridged12
- added C12, C13: 100nF, 0-Footprints:C_Disc_D5.0mm_W2.5mm_P5.00mm, symbol Device:C
- added U8, U9: 74LS245, 0-Footprints:DIP-20_W7.62mm, symbol 74xx:74LS245
Connections:
- net ~{BANK_{HB}} is gone; now on net ~{CS_RAM_{HB}}: U7.6 (~{CEO})
- net ~{BANK_{LB}} is gone; now on net ~{CS_RAM_{LB}}: U6.6 (~{CEO})
- net +5V: now also C12.1, C13.1, U8.1 (A->B), U8.20 (VCC), U9.1 (A->B), U9.20 (VCC)
- net +5V_{HB}: now also C2.1, U2.32 (VCC)
- net +5V_{LB}: now also C1.1, U1.32 (VCC)
- net BANK_0: now also U8.18 (B0), U9.18 (B0); no longer U3.12 (Q7), U5.12 (Q7)
- net BANK_1: now also U8.17 (B1), U9.17 (B1); no longer U3.13 (Q6), U5.13 (Q6)
- net BANK_2: now also U8.16 (B2), U9.16 (B2); no longer U3.14 (Q5), U5.14 (Q5)
- net BANK_3: now also U8.15 (B3), U9.15 (B3); no longer U3.15 (Q4), U5.15 (Q4)
- net BANK_4: now also U8.14 (B4), U9.14 (B4); no longer U3.16 (Q3), U5.16 (Q3)
- net BANK_5: now also U8.13 (B5), U9.13 (B5); no longer U3.17 (Q2), U5.17 (Q2)
- net BANK_6: now also U8.12 (B6), U9.12 (B6); no longer U3.18 (Q1), U5.18 (Q1)
- net BANK_7: now also U8.11 (B7), U9.11 (B7); no longer U3.19 (Q0), U5.19 (Q0)
- net D0: now also U3.2 (D0), U5.2 (D0); no longer U3.9 (D7), U5.9 (D7)
- net D1: now also U3.3 (D1), U5.3 (D1); no longer U3.8 (D6), U5.8 (D6)
- net D2: now also U3.4 (D2), U5.4 (D2); no longer U3.7 (D5), U5.7 (D5)
- net D3: now also U3.5 (D3), U5.5 (D3); no longer U3.6 (D4), U5.6 (D4)
- net D4: now also U3.6 (D4), U5.6 (D4); no longer U3.5 (D3), U5.5 (D3)
- net D5: now also U3.7 (D5), U5.7 (D5); no longer U3.4 (D2), U5.4 (D2)
- net D6: now also U3.8 (D6), U5.8 (D6); no longer U3.3 (D1), U5.3 (D1)
- net D7: now also U3.9 (D7), U5.9 (D7); no longer U3.2 (D0), U5.2 (D0)
- net GND: now also U3.1 (OE), U5.1 (OE), C12.2, C13.2, U8.10 (GND), U9.10 (GND); no longer U4.15 (I/O), U4.16 (I/O)
- net LOAD_{H}: now also U4.15 (I/O); no longer U4.19 (I/O)
- net LOAD_{L}: now also U4.16 (I/O); no longer U4.20 (I/O)
- net ~{OE}: now also U4.18 (I/O); no longer U4.22 (I/O)
- net ~{WE}: now also U4.17 (I/O); no longer U4.21 (I/O)
- net ~{CS_RAM_{LB}}: now reaches U1.22 (CE#)
- net ~{CS_RAM_{HB}}: now reaches U2.22 (CE#)
- removed net ~{BANK_{H}}: U3.1 (OE), U4.17 (I/O), U7.5 (~{CE})
- removed net ~{BANK_{L}}: U4.18 (I/O), U5.1 (OE), U6.5 (~{CE})
- new net: U5.19 (Q0), U8.2 (A0)
- new net: U5.18 (Q1), U8.3 (A1)
- new net: U5.17 (Q2), U8.4 (A2)
- new net: U5.16 (Q3), U8.5 (A3)
- new net: U5.15 (Q4), U8.6 (A4)
- new net: U5.14 (Q5), U8.7 (A5)
- new net: U5.13 (Q6), U8.8 (A6)
- new net: U3.13 (Q6), U9.8 (A6)
- new net: U3.14 (Q5), U9.7 (A5)
- new net: U3.15 (Q4), U9.6 (A4)
- new net: U3.16 (Q3), U9.5 (A3)
- new net: U3.17 (Q2), U9.4 (A2)
- new net: U3.18 (Q1), U9.3 (A1)
- new net: U3.19 (Q0), U9.2 (A0)
- new net LATCH_BANK7_H: U3.12 (Q7), U4.21 (I/O), U9.9 (A7)
- new net LATCH_BANK7_L: U4.22 (I/O), U5.12 (Q7), U8.9 (A7)
- new net ~{CS_H}: U9.19 (CE)
- new net ~{CS_L}: U8.19 (CE)
- new net ~{CS_RAM_{H}}: U4.19 (I/O), U7.5 (~{CE})
- new net ~{CS_RAM_{L}}: U4.20 (I/O), U6.5 (~{CE})
Other:
- note added: "~{OE}: BUS_OK && !~{BANK_SEL} && R/~{W} ~{WE}: BUS_OK && !~{BANK_SEL} && !R/~{W} LOAD_{L}: BUS_OK && !~{IO_SEL} && !A0 && ![A1..A7] && !R/~{W} LOAD_{H}: BUS_OK && !~{IO_SEL} && A0 && ![A1..A7] && !R/~{W} SEL_BANK7 = (!A12 & LATCH_BANK7_L) # (A12 & LATCH_BANK7_H) ~{CS_RAM_{L}}: !(BUS_OK && !~{BANK_SEL} && SEL_BANK7) ~{CS_RAM_{H}}: !(BUS_OK && !~{BANK_SEL} && !SEL_BANK7)"
- note removed: "~{OE}: BUS_OK && !~{BANK_SEL} && R/~{W} ~{WE}: BUS_OK && !~{BANK_SEL} && !R/~{W} LOAD_{L}: BUS_OK && !~{IO_SEL} && !A0 && ![A1..A7] && !R/~{W} LOAD_{H}: BUS_OK && !~{IO_SEL} && A0 && ![A1..A7] && !R/~{W} ~{BANK_{L}}: BUS_OK && !~{IO_SEL} & !A12 ~{BANK_{H}}: BUS_OK && !~{IO_SEL} & A12"
- moved on the sheet: C1, C2, C3, C5, U1, U2, U3, U4
