File: Front/Faceplate/Faceplate.kicad_pcb (KiCad board)
At the start: 2 copper layers, 200.2 x 100 mm, 74 parts, among them SW1 D0, SW10 A1, SW11 A2, SW12 A3, SW13 A4, SW14 A5, SW15 A6, SW16 A7, SW17 A8, SW18 A9, SW19 A10, SW2 D1, SW20 A11, SW21 A12, SW22 A13, SW23 A14, SW24 A15, SW25 POWER, SW26 RESET, SW3 D2, SW4 D3, SW5 D4, SW6 D5, SW7 D6, SW8 D7, SW9 A0

Commit message: lots of fixes to stack handling on emu, fix the latches on the banked memory board, tons of little bug fixes
Other:
- board size 200.2 x 100 mm -> 328.4 x 100 mm
